File: temperature_controller_2.sch (KiCad schematic (older format))
At the start: 6 parts

Commit message: Added 2.5V referece.
Parts:
- added C?: 0.1uF, symbol C
- added C? (x2): 1uF, symbol C
- added U?: AD780, symbol AD780
Connections:
- net +15V: now also C?.1, C?.2, U?.2 (+VIN)
- net GND: now reaches C?.1, C?.2, C?.2, U?.2 (GND)
- net GND: now also C?.1, C?.2, C?.2, U?.4 (GND)
- new net 2.5V: C?.1, U?.6 (VOUT)
- no-connect marks 0 -> 5
Changed lines of the file:
@@
 	2450 1750 2450 1800
 Connection ~ 2450 1750
+$Comp
+L AD780 U?
+U 1 1 58FA5755
+P 4600 1350
+F 0 "U?" H 4600 950 60  0000 C CNN
+F 1 "AD780" H 4600 1650 60  0000 C CNN
+F 2 "" H 4550 1200 60  0000 C CNN
+F 3 "" H 4550 1200 60  0000 C CNN
+	1    4600 1350
+	1    0    0    -1
+$EndComp
+$Comp
+L +15V #PWR?
+U 1 1 58FA57C4
+P 3950 1300
+F 0 "#PWR?" H 3950 1150 50  0001 C CNN
+F 1 "+15V" H 3950 1440 50  0000 C CNN
+F 2 "" H 3950 1300 50  0001 C CNN
+F 3 "" H 3950 1300 50  0001 C CNN
+	1    3950 1300
+	1    0    0    -1
+$EndComp
+Wire Wire Line
+	3350 1300 4150 1300
+$Comp
+L C C?
+U 1 1 58FA5813
+P 3650 1450
+F 0 "C?" H 3500 1350 50  0000 L CNN
+F 1 "0.1uF" H 3400 1550 50  0000 L CNN
+F 2 "" H 3688 1300 50  0001 C CNN
+F 3 "" H 3650 1450 50  0001 C CNN
+	1    3650 1450
+	-1   0    0    1
+$EndComp
+Connection ~ 3950 1300
+$Comp
+L C C?
+U 1 1 58FA58BC
+P 3350 1450
+F 0 "C?" H 3375 1550 50  0000 L CNN
+F 1 "1uF" H 3375 1350 50  0000 L CNN
+F 2 "" H 3388 1300 50  0001 C CNN
+F 3 "" H 3350 1450 50  0001 C CNN
+	1    3350 1450
+	1    0    0    -1
+$EndComp
+Wire Wire Line
+	3350 1600 4150 1600
+Connection ~ 3650 1600
+Connection ~ 3650 1300
+$Comp
+L GND #PWR?
+U 1 1 58FA59BE
+P 1750 1450
+F 0 "#PWR?" H 1750 1200 50  0001 C CNN
+F 1 "GND" H 1750 1300 50  0000 C CNN
+F 2 "" H 1750 1450 50  0001 C CNN
+F 3 "" H 1750 1450 50  0001 C CNN
+	1    1750 1450
+	1    0    0    -1
+$EndComp
+Wire Wire Line
+	1750 1350 1750 1450
+Connection ~ 1750 1350
+$Comp
+L PWR_FLAG #FLG?
+U 1 1 58FA5A1F
+P 1800 1250
+F 0 "#FLG?" H 1800 1325 50  0001 C CNN
+F 1 "PWR_FLAG" H 1800 1400 50  0000 C CNN
+F 2 "" H 1800 1250 50  0001 C CNN
+F 3 "" H 1800 1250 50  0001 C CNN
+	1    1800 1250
+	1    0    0    -1
+$EndComp
+Wire Wire Line
+	1800 1250 1800 1350
+Connection ~ 1800 1350
+$Comp
+L PWR_FLAG #FLG?
+U 1 1 58FA5A69
+P 1650 2000
+F 0 "#FLG?" H 1650 2075 50  0001 C CNN
+F 1 "PWR_FLAG" H 1650 2150 50  0000 C CNN
+F 2 "" H 1650 2000 50  0001 C CNN
+F 3 "" H 1650 2000 50  0001 C CNN
+	1    1650 2000
+	1    0    0    -1
+$EndComp
+Wire Wire Line
+	1650 2000 1850 2000
+Wire Wire Line
+	1850 2000 1850 1750
+Connection ~ 1850 1750
+NoConn ~ 4150 1450
+NoConn ~ 5050 1150
+NoConn ~ 5050 1300
+NoConn ~ 4150 1150
+$Comp
+L C C?
+U 1 1 58FA5B83
+P 5300 1600
+F 0 "C?" H 5325 1700 50  0000 L CNN
+F 1 "1uF" H 5325 1500 50  0000 L CNN
+F 2 "" H 5338 1450 50  0001 C CNN
+F 3 "" H 5300 1600 50  0001 C CNN
+	1    5300 1600
+	1    0    0    -1
+$EndComp
+Wire Wire Line
+	5050 1450 5300 1450
+$Comp
+L GND #PWR?
+U 1 1 58FA5C1C
+P 3900 1700
+F 0 "#PWR?" H 3900 1450 50  0001 C CNN
+F 1 "GND" H 3900 1550 50  0000 C CNN
+F 2 "" H 3900 1700 50  0001 C CNN
+F 3 "" H 3900 1700 50  0001 C CNN
+	1    3900 1700
+	1    0    0    -1
+$EndComp
+Wire Wire Line
+	3900 1600 3900 1700
+Connection ~ 3900 1600
+$Comp
+L GND #PWR?
+U 1 1 58FA5C77
+P 5300 1800
+F 0 "#PWR?" H 5300 1550 50  0001 C CNN
+F 1 "GND" H 5300 1650 50  0000 C CNN
+F 2 "" H 5300 1800 50  0001 C CNN
+F 3 "" H 5300 1800 50  0001 C CNN
+	1    5300 1800
+	1    0    0    -1
+$EndComp
+Wire Wire Line
+	5300 1750 5300 1800
+NoConn ~ 5050 1600
+Text Label 5300 1350 0    60   ~ 0
+2.5V
+Wire Wire Line
+	5300 1450 5300 1350
 $EndSCHEMATC

Commit message: Schematic completed.
Parts:
- added C? (x3): 10uF, symbol C
- added C? (x10): 0.1uF, symbol C
- added C? (x2): 1uF, symbol C
- added C?: 10000pF, symbol C
- added C?: 0.022uF, symbol C
- added C?: 22uF, symbol C
- added C?: 47uF, symbol C
- added C?: 330pF, symbol C
- added P? (x2): Ext. Mod./Monitor, symbol Dual-BNC
- added Q?: IRF540N, TO_SOT_Packages_THT:TO-220_Vertical, symbol IRF540N
- added Q?: IRF9540N, TO_SOT_Packages_THT:TO-220_Vertical, symbol IRF9540N
- added R? (x2): 5.1k, symbol R
- added R? (x12): 10k, symbol R
- added R? (x4): 1k, symbol R
- added R? (x5): 100k, symbol R
- added R?: 33k, symbol R
- added R?: 3.3k, symbol R
- added R?: 511, symbol R
- added R?: 330k, symbol R
- added R?: 100, symbol R
- added R?: 12, symbol R
- added R? (x2): 200k, symbol R
- added R?: 0.5, symbol R
- added RV?: 10k, symbol POT
- added S? (x8): spdt, symbol spdt
- added TP? (x7): TEST, symbol TEST
- added U? (x2): R_th, symbol ED2580
- added U? (x2): 8DIP, symbol 8DIP
- added U?: INA188, symbol INA188
- added U? (x8): OP497, symbol OP497
Connections:
- net +15V: now also C?.2, C?.2, C?.2, Q?.2 (D), U?.4 (V+), U?.4 (V+), U?.7 (V+)
- net -15V: now also C?.2, C?.2, C?.2, Q?.2 (D), U?.13 (V-), U?.13 (V-), U?.4 (V-)
- net 2.5V: now also R?.1, R?.1, TP?.1
- net GND: now also C?.1, C?.1, C?.1, C?.1, C?.1, C?.1, C?.1, C?.1, C?.2, C?.2, P?.2, P?.4, R?.1, R?.1, R?.2, R?.2, R?.2, S?.3, U?.14 (+), U?.14 (+), U?.2, U?.2, U?.3 (+), U?.5 (+), U?.5 (REF)
- new net: R?.2, RV?.1
- new net: R?.1, RV?.3
- new net: S?.1, U?.1
- new net: R?.1, S?.3
- new net: R?.1, U?.1, U?.15 (-), U?.2, U?.3, U?.4, U?.5, U?.6, U?.7, U?.8
- new net: R?.2, U?.10
- new net: R?.2, U?.11
- new net: R?.2, U?.12
- new net: R?.2, U?.13
- new net: R?.2, U?.14
- new net: R?.2, U?.15
- new net: R?.2, U?.16
- new net: R?.2, U?.9
- new net: S?.2, S?.3
- new net: R?.2, U?.1 (RG)
- new net: R?.2, TP?.1, U?.6 (VOUT)
- new net: R?.1, U?.8 (RG)
- new net: R?.1, R?.1, R?.1, R?.1, R?.1, R?.1, R?.1, R?.1, R?.2, U?.16
- new net: C?.2, R?.1, R?.1, R?.2, U?.2 (-)
- new net: R?.1, U?.5 (+)
- new net: P?.3, U?.6 (-), U?.7
- new net: C?.1, R?.1, S?.1, S?.2, U?.10
- new net: C?.2, R?.2, R?.2, S?.3, U?.11 (-)
- new net: R?.1, R?.2, S?.3, U?.1
- new net: R?.1, S?.3, U?.1, U?.2, U?.2 (-), U?.3, U?.4, U?.5, U?.6, U?.7, U?.8
- new net: U?.6 (-), U?.7
- new net: C?.1, R?.2, U?.10
- new net: R?.1, R?.1, R?.2, U?.11 (-)
- new net: R?.1, R?.1, U?.12 (+)
- new net: R?.1, R?.2, U?.15 (-)
- new net: R?.2, S?.1, U?.16
- new net: R?.2, S?.2
- new net: P?.1, R?.2
- new net: C?.2, U?.10
- new net: C?.2, U?.11
- new net: C?.2, U?.12
- new net: C?.2, U?.13
- new net: C?.2, U?.14
- new net: C?.2, U?.16
- new net: C?.1, C?.1, C?.1, C?.1, C?.1, C?.1, R?.1, S?.2, U?.9
- new net: S?.1, S?.2
- new net: Q?.1 (G), Q?.1 (G), R?.1, R?.2
- new net: Q?.3 (S), S?.1
- new net: C?.2, R?.1
- new net Rs+: Q?.3 (S), R?.1, R?.2, S?.2, TP?.1
- new net Rs-: R?.2, R?.2, TP?.1, U?.1
- new net act_t: C?.1, C?.2, R?.2, S?.1, S?.2, TP?.1, U?.3 (VIN+)
- new net error_signal: C?.1, R?.1, R?.2, TP?.1, U?.1, U?.12 (+)
- new net set_t: C?.1, C?.2, RV?.2, S?.3, TP?.1, U?.2 (VIN-)
- new net v_servo: R?.2, S?.2
- no-connect marks 5 -> 6
Other:
- note added: "30 Hz LP filter on act_t"
- note added: "3Hz LP filter on set_t"
- note added: "I_load = -v_servo*(10k/200k)/R_sense\nI_load (A) = v_servo(V)/10\nI_load (A) < 15/10 = 1.5A"
- note added: "PI Pole (Hz)\n72\n16\n1.6\n0.16\n0.16\n0.07\n0.04\nOff\n\n\n"
- note added: "Precision low noise 2.5V reference"
- note added: "Wheatstone bridge for thermister resistance measurement.\nSwitch to internal low tempco resistor for measuring opamp noise"
- note added: "error_signal has a nominal change of 6.25 V/K at 25C.\nError signal monitor has a flip switch for monitoring \nerror_signal or 101x error signal"
- note added: "gains\n100\n33\n10\n3.3\n1\n0.33\n0.1\n0"

Commit message: Footprints assigned.
Parts:
- C1, C10, C11, C12, C13, C14, C15, C16, C17, C18, C19, C2, C20, C21, C22, C24, C25, C27, C28, C3, C4, C5, C6, C7, C8, C9: renamed from C?; footprint (none) -> Capacitors_SMD:C_0603_HandSoldering
- C23: renamed from C?; value 47uF -> 22uF; footprint (none) -> Capacitors_SMD:C_1206_HandSoldering
- C26: renamed from C?; footprint (none) -> Capacitors_SMD:C_1206_HandSoldering
- P1: renamed from P?; footprint (none) -> local_footprints:Dual-BNC-ARF2136
- R1, R10, R11, R13, R14, R15, R16, R17, R18, R19, R2, R20, R21, R22, R23, R24, R25, R26, R27, R28, R29, R3, R30, R31, R32, R4, R5, R6, R7, R8, R9: renamed from R?; footprint (none) -> Resistors_SMD:R_0603_HandSoldering
- R12: renamed from R?; footprint (none) -> Resistors_SMD:R_2512_HandSoldering
- RV1: renamed from RV?; footprint (none) -> local_footprints:VishaySpectrol536
- S1, S6, S7: renamed from S?; footprint (none) -> local_footprints:CJS-1200TB-SPDT
- S2, S3, S4, S5, S8: renamed from S?; footprint (none) -> local_footprints:SPDT-Horizontal
- TP1, TP2, TP3, TP4, TP5, TP6, TP7: renamed from TP?; footprint (none) -> Measurement_Points:Measurement_Point_Round-SMD-Pad_Small
- U1: renamed from U?; footprint (none) -> local_footprints:ED2610
- U2, U8: renamed from U?; footprint (none) -> Housings_SOIC:SOIC-16W_7.5x10.3mm_Pitch1.27mm
- U3, U5: renamed from U?; footprint (none) -> Housings_SOIC:SOIC-8_3.9x4.9mm_Pitch1.27mm
- U4, U9: renamed from U?; footprint (none) -> local_footprints:ED2580
- gave numbers to parts that had none: 4
Connections:
- net GND: now also U2.12 (+), U2.5 (+), U8.12 (+), U8.14 (+), U8.3 (+); no longer U2.14 (+), U2.3 (+), U8.14 (+), U8.5 (+)
- net error_signal: now also U2.14 (+), U2.7; no longer U2.1, U2.12 (+)
- net at R13.1, U6.1, U6.2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: now also U2.11 (-); no longer U2.15 (-)
- net at R16.1, R17.1, R18.1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: now also U2.10; no longer U2.16
- net at C9.2, R10.1, R11.2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: now also U2.6 (-); no longer U2.2 (-)
- net at C14.1, R15.1, S2.2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: now also U2.16; no longer U2.10
- net at C14.2, R14.2, R15.2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: now also U2.15 (-); no longer U2.11 (-)
- net at C1.1, R7.2: now also U2.1; no longer U2.10
- net at R1.1, R5.1, R6.2: now also U2.2 (-); no longer U2.11 (-)
- net at R3.1, R4.1: now also U2.3 (+); no longer U2.12 (+)
- net at R31.2, R32.1: now also U8.11 (-); no longer U8.15 (-)
- net at R32.2, S7.1: now also U8.10; no longer U8.16
- net at U7.15: now also C24.2
- net at C20.1, C21.1, C22.1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: now also C24.1
- new net: U8.15 (-), U8.16
- no-connect marks 6 -> 8
Other:
- note added: "PI Pole (Hz)\n72\n16\n1.6\n0.16\n0.16\n0.07\n0.07\nOff\n\n\n"
- note removed: "PI Pole (Hz)\n72\n16\n1.6\n0.16\n0.16\n0.07\n0.04\nOff\n\n\n"

Commit message: PCB component layout, first pass.
Parts:
- added J1: DB9_FEMALE, local_footprints:DB9_Throughhole, symbol DB9_FEMALE
- U4: value R_th -> Peltier/Heater
- U6, U7: footprint (none) -> local_footprints:8_POS_DIP_Switch
- renumbered U8 to U2, U2 to U8
Connections:
- net +15V: now also U8.4 (V+), J1.9; no longer U2.4 (V+)
- net -15V: now also U8.13 (V-), J1.8; no longer U2.13 (V-)
- net GND: now also U2.14 (+), U2.3 (+), U8.3 (+), J1.4, J1.5; no longer U2.12 (+), U2.3 (+), U8.14 (+)
- net error_signal: now also U2.12 (+); no longer U2.14 (+)
- net at R13.1, U6.1, U6.2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: now also U2.2 (-); no longer U2.11 (-)
- net at R16.1, R17.1, R18.1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: now also U2.1; no longer U2.10
- net at C14.2, R14.2, R15.2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: now also U2.11 (-); no longer U2.15 (-)
- net at C14.1, R15.1, S2.2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: now also U2.10; no longer U2.16
- net at R28.2, R31.1: now also S7.1, U2.16; no longer S7.3, U2.1
- net at R24.1, S4.3, U7.1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: now also U2.15 (-); no longer U2.2 (-)
- net at C1.1, R7.2: now also U8.16; no longer U8.1
- net at R1.1, R5.1, R6.2: now also U8.15 (-); no longer U8.2 (-)
- net at R3.1, R4.1: now also U8.14 (+); no longer U8.3 (+)
- net at R32.2, U8.10: now also S7.3; no longer S7.1
- new net: U8.1, U8.2 (-)
- no-connect marks 8 -> 13
Other:
- moved on the sheet: C18, C19, C2, C3, C6, C7, C8, U1
